Commit message: The robot slips because the mass and inertia values of the two wheels are unrealistic
Decrease them to fix the slipping.

File: mobile_robot/urdf/mobile_robot.xacro (robot description, xacro)
@@ -10,5 +10,5 @@
   <xacro:property name="wheel_radius" value="0.1"/>
   <xacro:property name="wheel_thickness" value="0.05"/>
-  <xacro:property name="wheel_mass" value="5.0"/>
+  <xacro:property name="wheel_mass" value="0.5"/>
   <!-- Wheel placement -->
   <xacro:property name="wheel_y_offset" value="${(chassis_width / 2) + (wheel_thickness / 2)}"/>
@@ -126,8 +126,8 @@
       <origin xyz="0 0 0" rpy="0 1.5707 1.5707"/>
       <mass value="${wheel_mass}"/>
-      <inertia ixx="0.1" ixy="0" ixz="0"
-               iyy="0.1" iyz="0"
-               izz="0.1"/>
-    </inertial>
+      <inertia ixx="0.00135" ixy="0" ixz="0"
+               iyy="0.00135" iyz="0"
+               izz="0.0025"/>
+      </inertial>
   </link>
   <joint type="continuous" name="left_wheel_joint">
@@ -156,7 +156,7 @@
       <origin xyz="0 0 0" rpy="0 1.5707 1.5707"/>
       <mass value="${wheel_mass}"/>
-      <inertia ixx="0.1" ixy="0" ixz="0"
-               iyy="0.1" iyz="0"
-               izz="0.1"/>
+      <inertia ixx="0.00135" ixy="0" ixz="0"
+               iyy="0.00135" iyz="0"
+               izz="0.0025"/>
     </inertial>
   </link>

Commit message: Add the generated xacro file from SolidWords

File: mobile_robot/urdf/mobile_robot.xacro (robot description, xacro)
@@ -1,198 +1,184 @@
-<?xml version="1.0"?>
+<?xml version='1.0'?>
 <robot name="mobile_robot" xmlns:xacro="http://www.ros.org/wiki/xacro">
-  <!-- ================== Parameters ================== -->
-  <!-- Chassis dimensions -->
-  <xacro:property name="chassis_length" value="0.4"/>
-  <xacro:property name="chassis_width"  value="0.2"/>
-  <xacro:property name="chassis_height" value="0.1"/>
-  <xacro:property name="chassis_mass"   value="15.0"/>
-  <!-- Wheel dimensions -->
-  <xacro:property name="wheel_radius" value="0.1"/>
-  <xacro:property name="wheel_thickness" value="0.05"/>
-  <xacro:property name="wheel_mass" value="0.5"/>
-  <!-- Wheel placement -->
-  <xacro:property name="wheel_y_offset" value="${(chassis_width / 2) + (wheel_thickness / 2)}"/>
-  <!-- Derived values -->
-  <xacro:property name="wheel_separation" value="${2 * wheel_y_offset}"/>
-  <xacro:property name="wheel_diameter" value="${2 * wheel_radius}"/>
-  <!-- Caster dimensions -->
-  <xacro:property name="caster_radius" value="0.05"/>
-  <xacro:property name="caster_z_offset" value="-0.05"/>
-  <xacro:property name="caster_front_x" value="0.15"/>
-  <xacro:property name="caster_rear_x"  value="-0.15"/>
-  <!-- Lidar dimensions -->
-  <xacro:property name="lidar_size" value="0.1"/>
-  <xacro:property name="lidar_x" value="0.15"/>
-  <xacro:property name="lidar_z" value="0.1"/>
-  <xacro:property name="lidar_mass" value="1e-5"/>
   <!-- ================== Includes ================== -->
   <xacro:include filename="$(find mobile_robot)/urdf/mobile_robot.gazebo" />
   <xacro:include filename="$(find mobile_robot)/urdf/materials.xacro" />
   <!--
-    Robot Structure:
-    - chassis (base)
-    - caster (front & rear)
-    - left_wheel_link
-    - right_wheel_link
-    - lidar_link
+    Robot Structure Overview:
+    - Chassis (base)
+    - 4 Casters (non-driven support wheels)
+    - Left & Right drive wheels
+    - Lidar sensor
   -->
-  <!-- ================== Base / Chassis ================== -->
+  <!-- ========================================================= -->
+  <!-- ================== Base / Chassis ======================= -->
+  <!-- ========================================================= -->
   <link name="chassis">
-    <pose>0 0 ${chassis_height/2} 0 0 0</pose>
     <!-- Inertia -->
     <inertial>
-      <mass value="${chassis_mass}"/>
-      <origin xyz="0 0 ${chassis_height/2}" rpy="0 0 0"/>
-      <inertia ixx="0.1" ixy="0" ixz="0"
-               iyy="0.1" iyz="0"
-               izz="0.1"/>
+      <mass value="56.8425142723701"/>
+      <origin xyz="0.000508426452289656 5.85230715788032E-05 0.532734267230434" rpy="0 0 0" />
+      <inertia
+        ixx="4.9887479320299" ixy="-0.000665021365264802" ixz="0.117153222467253"
+        iyy="3.29577614857709" iyz="9.17818860502157E-07"
+        izz="2.8376872224854" />
     </inertial>
-    <!-- Collision (box) -->
-    <collision name="chassis_collision">
+    <!-- Chassis Visual -->
+    <visual>
+      <origin xyz="0 0 0" rpy="0 0 0" />
       <geometry>
-        <box size="${chassis_length} ${chassis_width} ${chassis_height}"/>
+        <mesh filename="package://mobile_robot/meshes/chassis.STL" />
+      </geometry>
+      <material name="">
+        <color rgba="0.647058823529412 0.619607843137255 0.588235294117647 1" />
+      </material>
+    </visual>
+    <!-- Chassis Collision -->
+    <collision>
+      <origin xyz="0 0 0" rpy="0 0 0" />
+      <geometry>
+        <mesh filename="package://mobile_robot/meshes/chassis.STL" />
       </geometry>
     </collision>
-    <!-- Visual (box) -->
-    <visual name="chassis_visual">
-      <origin xyz="0 0 0" rpy="0 0 0"/>
-      <geometry>
-        <box size="${chassis_length} ${chassis_width} ${chassis_height}"/>
-      </geometry>
-    </visual>
-    <!-- Rear caster -->
-    <collision name="caster_rear_collision">
-      <origin xyz="${caster_rear_x} 0 ${caster_z_offset}" rpy="0 0 0"/>
-      <geometry>
-        <sphere radius="${caster_radius}"/>
-      </geometry>
+    <!-- ================== Casters (Support Spheres) ================== -->
+    <!-- Front Right Caster -->
+    <collision name='caster_1_collision'>
+      <origin xyz="0.165 0.09 0.031" rpy="0 0 0"/>
+      <geometry><sphere radius="0.03"/></geometry>
       <surface>
-        <friction>
-          <ode>
-            <mu>0</mu>
-            <mu2>0</mu2>
-            <slip1>1.0</slip1>
-            <slip2>1.0</slip2>
-          </ode>
-        </friction>
+        <friction><ode><mu>0</mu><mu2>0</mu2><slip1>1.0</slip1><slip2>1.0</slip2></ode></friction>
       </surface>
     </collision>
-    <visual name="caster_rear_visual">
-      <origin xyz="${caster_rear_x} 0 ${caster_z_offset}" rpy="0 0 0"/>
-      <geometry>
-        <sphere radius="${caster_radius}"/>
-      </geometry>
+    <visual name='caster_1_visual'>
+      <origin xyz="0.165 0.09 0.031" rpy="0 0 0"/>
+      <geometry><sphere radius="0.03"/></geometry>
     </visual>
-    <!-- Front caster -->
-    <collision name="caster_front_collision">
-      <origin xyz="${caster_front_x} 0 ${caster_z_offset}" rpy="0 0 0"/>
-      <geometry>
-        <sphere radius="${caster_radius}"/>
-      </geometry>
+    <!-- Front Left Caster -->
+    <collision name='caster_2_collision'>
+      <origin xyz="-0.165 0.09 0.031" rpy="0 0 0"/>
+      <geometry><sphere radius="0.03"/></geometry>
       <surface>
-        <friction>
-          <ode>
-            <mu>0</mu>
-            <mu2>0</mu2>
-            <slip1>1.0</slip1>
-            <slip2>1.0</slip2>
-          </ode>
-        </friction>
+        <friction><ode><mu>0</mu><mu2>0</mu2><slip1>1.0</slip1><slip2>1.0</slip2></ode></friction>
       </surface>
     </collision>
-    <visual name="caster_front_visual">
-      <origin xyz="${caster_front_x} 0 ${caster_z_offset}" rpy="0 0 0"/>
-      <geometry>
-        <sphere radius="${caster_radius}"/>
-      </geometry>
+    <visual name='caster_2_visual'>
+      <origin xyz="-0.165 0.09 0.031" rpy="0 0 0"/>
+      <geometry><sphere radius="0.03"/></geometry>
+    </visual>
+    <!-- Rear Right Caster -->
+    <collision name='caster_3_collision'>
+      <origin xyz="0.165 -0.09 0.031" rpy="0 0 0"/>
+      <geometry><sphere radius="0.03"/></geometry>
+      <surface>
+        <friction><ode><mu>0</mu><mu2>0</mu2><slip1>1.0</slip1><slip2>1.0</slip2></ode></friction>
+      </surface>
+    </collision>
+    <visual name='caster_3_visual'>
+      <origin xyz="0.165 -0.09 0.031" rpy="0 0 0"/>
+      <geometry><sphere radius="0.03"/></geometry>
+    </visual>
+    <!-- Rear Left Caster -->
+    <collision name='caster_4_collision'>
+      <origin xyz="-0.165 -0.09 0.031" rpy="0 0 0"/>
+      <geometry><sphere radius="0.03"/></geometry>
+      <surface>
+        <friction><ode><mu>0</mu><mu2>0</mu2><slip1>1.0</slip1><slip2>1.0</slip2></ode></friction>
+      </surface>
+    </collision>
+    <visual name='caster_4_visual'>
+      <origin xyz="-0.165 -0.09 0.031" rpy="0 0 0"/>
+      <geometry><sphere radius="0.03"/></geometry>
     </visual>
   </link>
   <!-- ================== End Chassis ================== -->
-  <!-- ================== Left Wheel ================== -->
+  <!-- ========================================================= -->
+  <!-- ================== Left Wheel ========================== -->
+  <!-- ========================================================= -->
   <link name="left_wheel_link">
-    <collision name="left_wheel_collision">
-      <origin xyz="0 0 0" rpy="0 1.5707 1.5707"/>
-      <geometry>
-        <cylinder radius="${wheel_radius}" length="${wheel_thickness}"/>
-      </geometry>
+    <gravity>1</gravity>
+    <inertial>
+      <origin xyz="0 0 0" rpy="0 0 0" />
+      <mass value="0.238183102723088" />
+      <inertia
+        ixx="0.000429468568590385" ixy="2.82194133801453E-08" ixz="3.45307405175469E-09"
+        iyy="0.000813895351440581" iyz="9.00820636504668E-09"
+        izz="0.000429448713932949" />
+    </inertial>
+    <visual>
+      <origin xyz="0 0 0" rpy="0 0 0" />
+      <geometry><mesh filename="package://mobile_robot/meshes/left_wheel_link.STL" /></geometry>
+      <material name=""><color rgba="0 0 0 1" /></material>
+    </visual>
+    <collision>
+      <origin xyz="0 0 0" rpy="0 0 0" />
+      <geometry><mesh filename="package://mobile_robot/meshes/left_wheel_link.STL" /></geometry>
     </collision>
-    <visual name="left_wheel_visual">
-      <origin xyz="0 0 0" rpy="0 1.5707 1.5707"/>
-      <geometry>
-        <cylinder radius="${wheel_radius}" length="${wheel_thickness}"/>
-      </geometry>
+  </link>
+  <!-- Left Wheel Joint -->
+  <joint name="left_wheel_joint" type="continuous">
+    <origin xyz="0.0047501 0.241 0.073998" rpy="0 0 0" />
+    <parent link="chassis" />
+    <child link="left_wheel_link" />
+    <axis xyz="0 1 0" />
+    <limit effort="10000" velocity="100" />
+    <dynamics damping="1" friction="1" />
+  </joint>
+  <!-- ========================================================= -->
+  <!-- ================== Right Wheel ========================= -->
+  <!-- ========================================================= -->
+  <link name="right_wheel_link">
+    <gravity>1</gravity>
+    <inertial>
+      <origin xyz="0 0 0" rpy="0 0 0" />
+      <mass value="0.238183102723089" />
+      <inertia
+        ixx="0.000429448212823663" ixy="5.93719116295323E-09" ixz="-1.22691894940822E-09"
+        iyy="0.000813895360705823" iyz="-2.90318197452589E-08"
+        izz="0.000429469050110622" />
+    </inertial>
+    <visual>
+      <origin xyz="0 0 0" rpy="0 0 0" />
+      <geometry><mesh filename="package://mobile_robot/meshes/right_wheel_link.STL" /></geometry>
+      <material name=""><color rgba="0.792156862745098 0.819607843137255 0.933333333333333 1" /></material>
     </visual>
+    <collision>
+      <origin xyz="0 0 0" rpy="0 0 0" />
+      <geometry><mesh filename="package://mobile_robot/meshes/right_wheel_link.STL" /></geometry>
+    </collision>
+  </link>
+  <!-- Right Wheel Joint -->
+  <joint name="right_wheel_joint" type="continuous">
+    <origin xyz="0.0049293 -0.235 0.074053" rpy="0 0 0" />
+    <parent link="chassis" />
+    <child link="right_wheel_link" />
+    <axis xyz="0 1 0" />
+    <limit effort="10000" velocity="100" />
+    <dynamics damping="1" friction="1" />
+  </joint>
+  <!-- ========================================================= -->
+  <!-- ================== Lidar Sensor ======================== -->
+  <!-- ========================================================= -->
+  <link name="lidar_link">
     <inertial>
-      <origin xyz="0 0 0" rpy="0 1.5707 1.5707"/>
-      <mass value="${wheel_mass}"/>
-      <inertia ixx="0.00135" ixy="0" ixz="0"
-               iyy="0.00135" iyz="0"
-               izz="0.0025"/>
-      </inertial>
+      <origin xyz="0 0 0" rpy="0 0 0" />
+      <mass value="0" />
+      <inertia ixx="0" ixy="0" ixz="0" iyy="0" iyz="0" izz="0" />
+    </inertial>
+    <visual>
+      <origin xyz="0 0 0" rpy="0 0 0" />
+      <geometry><mesh filename="package://mobile_robot/meshes/lidar.STL" /></geometry>
+      <material name=""><color rgba="1 1 1 1" /></material>
+    </visual>
+    <collision>
+      <origin xyz="0 0 0" rpy="0 0 0" />
+      <geometry><mesh filename="package://mobile_robot/meshes/lidar.STL" /></geometry>
+    </collision>
   </link>
-  <joint type="continuous" name="left_wheel_joint">
-    <origin xyz="0 ${wheel_y_offset} 0" rpy="0 0 0"/>
-    <child link="left_wheel_link"/>
-    <parent link="chassis"/>
-    <axis xyz="0 1 0"/>
-    <limit effort="10000" velocity="1000"/>
-  </joint>
-  <!-- ================== End Left Wheel ================== -->
-  <!-- ================== Right Wheel ================== -->
-  <link name="right_wheel_link">
-    <collision name="right_wheel_collision">
-      <origin xyz="0 0 0" rpy="0 1.5707 1.5707"/>
-      <geometry>
-        <cylinder radius="${wheel_radius}" length="${wheel_thickness}"/>
-      </geometry>
-    </collision>
-    <visual name="right_wheel_visual">
-      <origin xyz="0 0 0" rpy="0 1.5707 1.5707"/>
-      <geometry>
-        <cylinder radius="${wheel_radius}" length="${wheel_thickness}"/>
-      </geometry>
-    </visual>
-    <inertial>
-      <origin xyz="0 0 0" rpy="0 1.5707 1.5707"/>
-      <mass value="${wheel_mass}"/>
-      <inertia ixx="0.00135" ixy="0" ixz="0"
-               iyy="0.00135" iyz="0"
-               izz="0.0025"/>
-    </inertial>
-  </link>
-  <joint type="continuous" name="right_wheel_joint">
-    <origin xyz="0 -${wheel_y_offset} 0" rpy="0 0 0"/>
-    <child link="right_wheel_link"/>
-    <parent link="chassis"/>
-    <axis xyz="0 1 0"/>
-    <limit effort="10000" velocity="1000"/>
-  </joint>
-  <!-- ================== End Right Wheel ================== -->
-  <!-- ================== Lidar ================== -->
-  <link name="lidar_link">
-    <collision name="lidar_collision">
-      <origin xyz="0 0 0" rpy="0 0 0"/>
-      <geometry>
-        <box size="${lidar_size} ${lidar_size} ${lidar_size}"/>
-      </geometry>
-    </collision>
-    <visual name="lidar_visual">
-      <origin xyz="0 0 0" rpy="0 0 0"/>
-      <geometry>
-        <box size="${lidar_size} ${lidar_size} ${lidar_size}"/>
-      </geometry>
-    </visual>
-    <inertial>
-      <mass value="${lidar_mass}"/>
-      <origin xyz="0 0 0" rpy="0 0 0"/>
-      <inertia ixx="1e-6" ixy="0" ixz="0"
-               iyy="1e-6" iyz="0"
-               izz="1e-6"/>
-    </inertial>
-  </link>
+  <!-- Lidar Joint -->
   <joint name="lidar_joint" type="fixed">
-    <origin xyz="${lidar_x} 0 ${lidar_z}" rpy="0 0 0"/>
-    <parent link="chassis"/>
-    <child link="lidar_link"/>
+    <origin xyz="0.265061370158194 -0.000471092424494723 0.0889500000000105" rpy="0 0 0" />
+    <parent link="chassis" />
+    <child link="lidar_link" />
+    <axis xyz="0 0 0" />
   </joint>
   <!-- ================== End Lidar ================== -->
