Commit message: Declare link for 4 casters

File: mobile_robot/urdf/mobile_robot.xacro (robot description, xacro)
@@ -7,5 +7,5 @@
     Robot Structure Overview:
     - Chassis (base)
-    - 4 Casters (non-driven support wheels)
+    - 4 Caster links (non-driven support wheels)
     - Left & Right drive wheels
     - Lidar sensor
@@ -15,170 +15,150 @@
   <!-- ========================================================= -->
   <link name="chassis">
-    <!-- Inertia -->
     <inertial>
-      <mass value="56.8425142723701"/>
-      <origin xyz="0.000508426452289656 5.85230715788032E-05 0.532734267230434" rpy="0 0 0" />
+      <mass value="30"/>
+      <origin xyz="0 0 0" rpy="0 0 0"/>
       <inertia
         ixx="4.9887479320299" ixy="-0.000665021365264802" ixz="0.117153222467253"
         iyy="3.29577614857709" iyz="9.17818860502157E-07"
-        izz="2.8376872224854" />
+        izz="2.8376872224854"/>
     </inertial>
     <!-- Chassis Visual -->
     <visual>
-      <origin xyz="0 0 0" rpy="0 0 0" />
-      <geometry>
-        <mesh filename="package://mobile_robot/meshes/chassis.STL" />
-      </geometry>
-      <material name="">
-        <color rgba="0.647058823529412 0.619607843137255 0.588235294117647 1" />
-      </material>
+      <origin xyz="0 0 0" rpy="0 0 0"/>
+      <geometry><mesh filename="package://mobile_robot/meshes/chassis.STL"/></geometry>
+      <material name=""><color rgba="0.647 0.620 0.588 1"/></material>
     </visual>
     <!-- Chassis Collision -->
     <collision>
-      <origin xyz="0 0 0" rpy="0 0 0" />
-      <geometry>
-        <mesh filename="package://mobile_robot/meshes/chassis.STL" />
-      </geometry>
+      <origin xyz="0 0 0" rpy="0 0 0"/>
+      <geometry><mesh filename="package://mobile_robot/meshes/chassis.STL"/></geometry>
     </collision>
-    <!-- ================== Casters (Support Spheres) ================== -->
-    <!-- Front Right Caster -->
-    <collision name='caster_1_collision'>
-      <origin xyz="0.165 0.09 0.031" rpy="0 0 0"/>
-      <geometry><sphere radius="0.03"/></geometry>
-      <surface>
-        <friction><ode><mu>0.2</mu><mu2>0.2</mu2><slip1>0</slip1><slip2>0.1</slip2></ode></friction>
-      </surface>
-    </collision>
-    <visual name='caster_1_visual'>
-      <origin xyz="0.165 0.09 0.031" rpy="0 0 0"/>
-      <geometry><sphere radius="0.03"/></geometry>
-    </visual>
-    <!-- Front Left Caster -->
-    <collision name='caster_2_collision'>
-      <origin xyz="-0.165 0.09 0.031" rpy="0 0 0"/>
-      <geometry><sphere radius="0.03"/></geometry>
-      <surface>
-        <friction><ode><mu>0.2</mu><mu2>0.2</mu2><slip1>0</slip1><slip2>0.1</slip2></ode></friction>
-      </surface>
-    </collision>
-    <visual name='caster_2_visual'>
-      <origin xyz="-0.165 0.09 0.031" rpy="0 0 0"/>
-      <geometry><sphere radius="0.03"/></geometry>
-    </visual>
-    <!-- Rear Right Caster -->
-    <collision name='caster_3_collision'>
-      <origin xyz="0.165 -0.09 0.031" rpy="0 0 0"/>
-      <geometry><sphere radius="0.03"/></geometry>
-      <surface>
-        <friction><ode><mu>0.2</mu><mu2>0.2</mu2><slip1>0</slip1><slip2>0.1</slip2></ode></friction>
-      </surface>
-    </collision>
-    <visual name='caster_3_visual'>
-      <origin xyz="0.165 -0.09 0.031" rpy="0 0 0"/>
-      <geometry><sphere radius="0.03"/></geometry>
-    </visual>
-    <!-- Rear Left Caster -->
-    <collision name='caster_4_collision'>
-      <origin xyz="-0.165 -0.09 0.031" rpy="0 0 0"/>
-      <geometry><sphere radius="0.03"/></geometry>
-      <surface>
-        <friction><ode><mu>0.2</mu><mu2>0.2</mu2><slip1>0</slip1><slip2>0.1</slip2></ode></friction>
-      </surface>
-    </collision>
-    <visual name='caster_4_visual'>
-      <origin xyz="-0.165 -0.09 0.031" rpy="0 0 0"/>
-      <geometry><sphere radius="0.03"/></geometry>
-    </visual>
   </link>
-  <!-- ================== End Chassis ================== -->
   <!-- ========================================================= -->
-  <!-- ================== Left Wheel ========================== -->
+  <!-- =============== Casters (Support Spheres) =============== -->
   <!-- ========================================================= -->
+  <!-- Caster Template -->
+  <xacro:macro name="caster" params="name x y z">
+    <link name="${name}_link">
+      <inertial>
+        <mass value="0.5"/>
+        <origin xyz="0 0 0"/>
+        <inertia ixx="0.00018" ixy="0" ixz="0"
+                 iyy="0.00018" iyz="0"
+                 izz="0.00018"/>
+      </inertial>
+      <visual>
+        <origin xyz="0 0 0" rpy="0 0 0"/>
+        <geometry><sphere radius="0.03"/></geometry>
+      </visual>
+      <collision>
+        <origin xyz="0 0 0" rpy="0 0 0"/>
+        <geometry><sphere radius="0.03"/></geometry>
+        <surface>
+          <friction>
+            <ode>
+              <mu>1.0</mu>
+              <mu2>1.0</mu2>
+              <slip1>0.01</slip1>
+              <slip2>0.01</slip2>
+            </ode>
+          </friction>
+        </surface>
+      </collision>
+    </link>
+    <joint name="${name}_joint" type="continuous">
+      <parent link="chassis"/>
+      <child link="${name}_link"/>
+      <origin xyz="${x} ${y} ${z}" rpy="0 0 0"/>
+      <axis xyz="0 0 1"/>
+    </joint>
+  </xacro:macro>
+  <!-- Instantiate 4 Casters -->
+  <xacro:caster name="caster_front_left"  x="-0.165" y="0.09"  z="0.031"/>
+  <xacro:caster name="caster_front_right" x="0.165"  y="0.09"  z="0.031"/>
+  <xacro:caster name="caster_rear_left"   x="-0.165" y="-0.09" z="0.031"/>
+  <xacro:caster name="caster_rear_right"  x="0.165"  y="-0.09" z="0.031"/>
+  <!-- ========================================================= -->
+  <!-- ======================== Wheels ========================= -->
+  <!-- ========================================================= -->
+  <!-- Left Wheel -->
   <link name="left_wheel_link">
-    <gravity>1</gravity>
     <inertial>
-      <origin xyz="0 0 0" rpy="0 0 0" />
-      <mass value="0.238183102723088" />
-      <inertia
-        ixx="0.000429468568590385" ixy="2.82194133801453E-08" ixz="3.45307405175469E-09"
-        iyy="0.000813895351440581" iyz="9.00820636504668E-09"
-        izz="0.000429448713932949" />
+      <mass value="0.238"/>
+      <origin xyz="0 0 0"/>
+      <inertia ixx="0.00043" ixy="0" ixz="0"
+               iyy="0.00081" iyz="0" izz="0.00043"/>
     </inertial>
     <visual>
-      <origin xyz="0 0 0" rpy="0 0 0" />
-      <geometry><mesh filename="package://mobile_robot/meshes/left_wheel_link.STL" /></geometry>
-      <material name=""><color rgba="0 0 0 1" /></material>
+      <origin xyz="0 0 0"/>
+      <geometry><mesh filename="package://mobile_robot/meshes/left_wheel_link.STL"/></geometry>
+      <material name=""><color rgba="0 0 0 1"/></material>
     </visual>
     <collision>
-      <origin xyz="0 0 0" rpy="0 0 0" />
-      <geometry><mesh filename="package://mobile_robot/meshes/left_wheel_link.STL" /></geometry>
+      <origin xyz="0 0 0"/>
+      <geometry><mesh filename="package://mobile_robot/meshes/left_wheel_link.STL"/></geometry>
     </collision>
   </link>
   <!-- Left Wheel Joint -->
   <joint name="left_wheel_joint" type="continuous">
-    <origin xyz="0.0047501 0.241 0.073998" rpy="0 0 0" />
-    <parent link="chassis" />
-    <child link="left_wheel_link" />
-    <axis xyz="0 1 0" />
-    <limit effort="10000" velocity="100" />
-    <dynamics damping="1" friction="1" />
+    <origin xyz="0 0.241 0.074" rpy="0 0 0"/>
+    <parent link="chassis"/>
+    <child link="left_wheel_link"/>
+    <axis xyz="0 1 0"/>
+    <limit effort="20000" velocity="2.5"/>
+    <dynamics damping="0.1" friction="1.0"/>
   </joint>
-  <!-- ========================================================= -->
-  <!-- ================== Right Wheel ========================= -->
-  <!-- ========================================================= -->
+  <!-- Right Wheel -->
   <link name="right_wheel_link">
-    <gravity>1</gravity>
     <inertial>
-      <origin xyz="0 0 0" rpy="0 0 0" />
-      <mass value="0.238183102723089" />
-      <inertia
-        ixx="0.000429448212823663" ixy="5.93719116295323E-09" ixz="-1.22691894940822E-09"
-        iyy="0.000813895360705823" iyz="-2.90318197452589E-08"
-        izz="0.000429469050110622" />
+      <mass value="0.238"/>
+      <origin xyz="0 0 0"/>
+      <inertia ixx="0.00043" ixy="0" ixz="0"
+               iyy="0.00081" iyz="0" izz="0.00043"/>
     </inertial>
     <visual>
-      <origin xyz="0 0 0" rpy="0 0 0" />
-      <geometry><mesh filename="package://mobile_robot/meshes/right_wheel_link.STL" /></geometry>
-      <material name=""><color rgba="0.792156862745098 0.819607843137255 0.933333333333333 1" /></material>
+      <origin xyz="0 0 0"/>
+      <geometry><mesh filename="package://mobile_robot/meshes/right_wheel_link.STL"/></geometry>
+      <material name=""><color rgba="0.79 0.82 0.93 1"/></material>
     </visual>
     <collision>
-      <origin xyz="0 0 0" rpy="0 0 0" />
-      <geometry><mesh filename="package://mobile_robot/meshes/right_wheel_link.STL" /></geometry>
+      <origin xyz="0 0 0"/>
+      <geometry><mesh filename="package://mobile_robot/meshes/right_wheel_link.STL"/></geometry>
     </collision>
   </link>
   <!-- Right Wheel Joint -->
   <joint name="right_wheel_joint" type="continuous">
-    <origin xyz="0.0049293 -0.235 0.074053" rpy="0 0 0" />
-    <parent link="chassis" />
-    <child link="right_wheel_link" />
-    <axis xyz="0 1 0" />
-    <limit effort="10000" velocity="100" />
-    <dynamics damping="1" friction="1" />
+    <origin xyz="0 -0.241 0.074" rpy="0 0 0"/>
+    <parent link="chassis"/>
+    <child link="right_wheel_link"/>
+    <axis xyz="0 1 0"/>
+    <limit effort="20000" velocity="2.5"/>
+    <dynamics damping="0.1" friction="1.0"/>
   </joint>
   <!-- ========================================================= -->
-  <!-- ================== Lidar Sensor ======================== -->
+  <!-- =================== Lidar Sensor ======================== -->
   <!-- ========================================================= -->
   <link name="lidar_link">
     <inertial>
-      <origin xyz="0 0 0" rpy="0 0 0" />
-      <mass value="0" />
-      <inertia ixx="0" ixy="0" ixz="0" iyy="0" iyz="0" izz="0" />
+      <mass value="0"/>
+      <origin xyz="0 0 0"/>
+      <inertia ixx="0" ixy="0" ixz="0" iyy="0" iyz="0" izz="0"/>
     </inertial>
     <visual>
-      <origin xyz="0 0 0" rpy="0 0 0" />
-      <geometry><mesh filename="package://mobile_robot/meshes/lidar.STL" /></geometry>
-      <material name=""><color rgba="1 1 1 1" /></material>
+      <origin xyz="0 0 0"/>
+      <geometry><mesh filename="package://mobile_robot/meshes/lidar.STL"/></geometry>
+      <material name=""><color rgba="1 1 1 1"/></material>
     </visual>
     <collision>
-      <origin xyz="0 0 0" rpy="0 0 0" />
-      <geometry><mesh filename="package://mobile_robot/meshes/lidar.STL" /></geometry>
+      <origin xyz="0 0 0"/>
+      <geometry><mesh filename="package://mobile_robot/meshes/lidar.STL"/></geometry>
     </collision>
   </link>
   <!-- Lidar Joint -->
   <joint name="lidar_joint" type="fixed">
-    <origin xyz="0.265061370158194 -0.000471092424494723 0.0889500000000105" rpy="0 0 0" />
-    <parent link="chassis" />
-    <child link="lidar_link" />
-    <axis xyz="0 0 0" />
+    <origin xyz="0.265 0 0.089" rpy="0 0 0"/>
+    <parent link="chassis"/>
+    <child link="lidar_link"/>
+    <axis xyz="0 0 0"/>
   </joint>
   <!-- ================== End Lidar ================== -->
