Commit message: Add IMU plugin for gazebo

File: mobile_robot_description/urdf/mobile_robot.gazebo.xacro (robot description, xacro)
@@ -80,4 +80,40 @@
     <pose>0 0 0 0 0 0</pose>
   </gazebo>
+  <!-- IMU sensor -->
+  <gazebo reference="imu_link">
+    <sensor type="imu" name="imu">
+      <always_on>true</always_on>
+      <visualize>true</visualize>
+    </sensor>
+    <material>Gazebo/FlatBlack</material>
+  </gazebo>
+  <gazebo>
+    <plugin name="imu_plugin" filename="libgazebo_ros_imu.so">
+      <alwaysOn>true</alwaysOn>
+      <bodyName>imu_link</bodyName>
+      <frameName>imu_link</frameName>
+      <topicName>imu</topicName>
+      <serviceName>imu_service</serviceName>
+      <gaussianNoise>0.0</gaussianNoise>
+      <updateRate>0</updateRate>
+      <imu>
+        <noise>
+          <type>gaussian</type>
+          <rate>
+            <mean>0.0</mean>
+            <stddev>2e-4</stddev>
+            <bias_mean>0.0000075</bias_mean>
+            <bias_stddev>0.0000008</bias_stddev>
+          </rate>
+          <accel>
+            <mean>0.0</mean>
+            <stddev>1.7e-2</stddev>
+            <bias_mean>0.1</bias_mean>
+            <bias_stddev>0.001</bias_stddev>
+          </accel>
+        </noise>
+      </imu>
+    </plugin>
+  </gazebo>
   <!-- LIDAR sensor -->
   <gazebo reference="lidar_link">

File: mobile_robot_description/urdf/mobile_robot.urdf.xacro (robot description, xacro)
@@ -137,4 +137,13 @@
   </joint>
   <!-- ========================================================= -->
+  <!-- =================== IMU Sensor ======================== -->
+  <!-- ========================================================= -->
+  <link name="imu_link"/>
+  <joint name="imu_joint" type="fixed">
+    <parent link="chassis"/>
+    <child link="imu_link"/>
+    <origin xyz="0 0 0.3" rpy="0 0 0"/>
+  </joint>
+  <!-- ========================================================= -->
   <!-- =================== Lidar Sensor ======================== -->
   <!-- ========================================================= -->

Commit message: Migrate IMU sensor to Gazebo Sim and fix world system plugins
- Replace libgazebo_ros_imu.so with native Gazebo Sim IMU sensor
- Add gz-sim-imu-system as a world-level plugin (not model-level)
- Explicitly load Physics, UserCommands, and SceneBroadcaster in
  world SDF to fix robot spawn service not being advertised

Test: gz topic -e -t /imu

File: mobile_robot_description/urdf/mobile_robot.gazebo.xacro (robot description, xacro)
@@ -72,39 +72,25 @@
     <pose>0 0 0 0 0 0</pose>
   </gazebo>
-  <!-- IMU sensor -->
+  <!-- IMU sensor (Gazebo Sim) -->
   <gazebo reference="imu_link">
-    <sensor type="imu" name="imu">
+    <sensor name="imu_sensor" type="imu">
       <always_on>true</always_on>
+      <update_rate>100</update_rate>
       <visualize>true</visualize>
+      <topic>imu</topic>
+      <gz_frame_id>imu_link</gz_frame_id>
+      <imu>
+        <angular_velocity>
+          <x><noise type="gaussian"><mean>0.0</mean><stddev>2e-4</stddev><bias_mean>0.0000075</bias_mean><bias_stddev>0.0000008</bias_stddev></noise></x>
+          <y><noise type="gaussian"><mean>0.0</mean><stddev>2e-4</stddev><bias_mean>0.0000075</bias_mean><bias_stddev>0.0000008</bias_stddev></noise></y>
+          <z><noise type="gaussian"><mean>0.0</mean><stddev>2e-4</stddev><bias_mean>0.0000075</bias_mean><bias_stddev>0.0000008</bias_stddev></noise></z>
+        </angular_velocity>
+        <linear_acceleration>
+          <x><noise type="gaussian"><mean>0.0</mean><stddev>1.7e-2</stddev><bias_mean>0.1</bias_mean><bias_stddev>0.001</bias_stddev></noise></x>
+          <y><noise type="gaussian"><mean>0.0</mean><stddev>1.7e-2</stddev><bias_mean>0.1</bias_mean><bias_stddev>0.001</bias_stddev></noise></y>
+          <z><noise type="gaussian"><mean>0.0</mean><stddev>1.7e-2</stddev><bias_mean>0.1</bias_mean><bias_stddev>0.001</bias_stddev></noise></z>
+        </linear_acceleration>
+      </imu>
     </sensor>
-    <material>Gazebo/FlatBlack</material>
-  </gazebo>
-  <gazebo>
-    <plugin name="imu_plugin" filename="libgazebo_ros_imu.so">
-      <alwaysOn>true</alwaysOn>
-      <bodyName>imu_link</bodyName>
-      <frameName>imu_link</frameName>
-      <topicName>imu</topicName>
-      <serviceName>imu_service</serviceName>
-      <gaussianNoise>0.0</gaussianNoise>
-      <updateRate>0</updateRate>
-      <imu>
-        <noise>
-          <type>gaussian</type>
-          <rate>
-            <mean>0.0</mean>
-            <stddev>2e-4</stddev>
-            <bias_mean>0.0000075</bias_mean>
-            <bias_stddev>0.0000008</bias_stddev>
-          </rate>
-          <accel>
-            <mean>0.0</mean>
-            <stddev>1.7e-2</stddev>
-            <bias_mean>0.1</bias_mean>
-            <bias_stddev>0.001</bias_stddev>
-          </accel>
-        </noise>
-      </imu>
-    </plugin>
   </gazebo>
   <!-- LIDAR sensor -->

Commit message: Migrate to Gazebo Sim gpu_lidar sensor
Remove deprecated gazebo_ros laser plugin (libgazebo_ros_laser.so)
and replace with gpu_lidar sensor type and gz-sim-sensors-system for ros_gz_sim compatibility

File: mobile_robot_description/urdf/mobile_robot.gazebo.xacro (robot description, xacro)
@@ -94,12 +94,14 @@
     </sensor>
   </gazebo>
-  <!-- LIDAR sensor -->
+  <!-- LiDAR sensor (Gazebo Sim) -->
   <gazebo reference="lidar_link">
-    <material>Gazebo/FlatBlack</material>
-    <sensor type="ray" name="lds_lfcd_sensor">
+    <sensor name='gpu_lidar' type='gpu_lidar'>
       <pose>0 0 0.02 0 0 0</pose>
+      <always_on>true</always_on>
       <visualize>true</visualize>
       <update_rate>5</update_rate>
-      <ray>
+      <topic>scan</topic>
+      <gz_frame_id>lidar_link</gz_frame_id>
+      <lidar>
         <scan>
           <horizontal>
@@ -120,9 +122,5 @@
           <stddev>0.01</stddev>
         </noise>
-      </ray>
-      <plugin name="gazebo_ros_lds_lfcd_controller" filename="libgazebo_ros_laser.so">
-        <topicName>/mobile_robot/laser/scan</topicName>
-        <frameName>lidar_link</frameName>
-      </plugin>
+      </lidar>
     </sensor>
   </gazebo>

Commit message: Support multi robo spawning
- New mobile_robot_multi package: reads robots.yaml and spawns N robots
  with per-robot RSP (frame_prefix), ros_gz_sim create, and namespaced
  cmd_vel/odom/imu/scan/joint_state bridges.
- Parameterize mobile_robot.gazebo.xacro with optional robot_name arg
  to prefix DiffDrive frames, sensor gz_frame_ids, and Gz topics.
  Default empty preserves single-robot behavior.

File: mobile_robot_description/urdf/mobile_robot.gazebo.xacro (robot description, xacro)
@@ -1,4 +1,9 @@
 <?xml version="1.0"?>
-<robot name="mobile_robot">
+<robot name="mobile_robot" xmlns:xacro="http://www.ros.org/wiki/xacro">
+  <!-- Multi-robot support: empty robot_name => no prefix (backwards compatible). -->
+  <xacro:arg name="robot_name" default=""/>
+  <xacro:property name="robot_name" value="$(arg robot_name)"/>
+  <xacro:property name="ns_topic" value="${('/' + robot_name) if robot_name else ''}"/>
+  <xacro:property name="ns_frame" value="${(robot_name + '/') if robot_name else ''}"/>
   <!-- Joint State Publisher — needed for robot_state_publisher to broadcast wheel/caster TF -->
   <gazebo>
@@ -15,8 +20,8 @@
       <wheel_separation>0.453</wheel_separation>
       <wheel_radius>0.072</wheel_radius>
-      <topic>cmd_vel</topic>
-      <odom_topic>odom</odom_topic>
-      <frame_id>odom</frame_id>
-      <child_frame_id>chassis</child_frame_id>
+      <topic>${ns_topic}/cmd_vel</topic>
+      <odom_topic>${ns_topic}/odom</odom_topic>
+      <frame_id>${ns_frame}odom</frame_id>
+      <child_frame_id>${ns_frame}chassis</child_frame_id>
       <max_linear_acceleration>1</max_linear_acceleration>
     </plugin>
@@ -83,6 +88,6 @@
       <update_rate>100</update_rate>
       <visualize>true</visualize>
-      <topic>imu</topic>
-      <gz_frame_id>imu_link</gz_frame_id>
+      <topic>${ns_topic}/imu</topic>
+      <gz_frame_id>${ns_frame}imu_link</gz_frame_id>
       <imu>
         <angular_velocity>
@@ -106,6 +111,6 @@
       <visualize>true</visualize>
       <update_rate>5</update_rate>
-      <topic>scan</topic>
-      <gz_frame_id>lidar_link</gz_frame_id>
+      <topic>${ns_topic}/scan</topic>
+      <gz_frame_id>${ns_frame}lidar_link</gz_frame_id>
       <lidar>
         <scan>
