Commit message: Split into sub packages/modules to manage the packages easier.

File: mobile_robot_description/urdf/mobile_robot.urdf.xacro (robot description, xacro)
@@ -1,7 +1,7 @@
 <?xml version='1.0'?>
-<robot name="mobile_robot" xmlns:xacro="http://www.ros.org/wiki/xacro">
+<robot name="mobile_robot_description" xmlns:xacro="http://www.ros.org/wiki/xacro">
   <!-- ================== Includes ================== -->
-  <xacro:include filename="$(find mobile_robot)/urdf/mobile_robot.gazebo" />
-  <xacro:include filename="$(find mobile_robot)/urdf/materials.xacro" />
+  <xacro:include filename="$(find mobile_robot_description)/urdf/mobile_robot.gazebo.xacro" />
+  <xacro:include filename="$(find mobile_robot_description)/urdf/materials.xacro" />
   <!--
     Robot Structure Overview:
@@ -26,5 +26,5 @@
     <visual>
       <origin xyz="0 0 0" rpy="0 0 0"/>
-      <geometry><mesh filename="package://mobile_robot/meshes/chassis.STL"/></geometry>
+      <geometry><mesh filename="package://mobile_robot_description/meshes/chassis.STL"/></geometry>
       <material name=""><color rgba="0.647 0.620 0.588 1"/></material>
     </visual>
@@ -32,5 +32,5 @@
     <collision>
       <origin xyz="0 0 0" rpy="0 0 0"/>
-      <geometry><mesh filename="package://mobile_robot/meshes/chassis.STL"/></geometry>
+      <geometry><mesh filename="package://mobile_robot_description/meshes/chassis.STL"/></geometry>
     </collision>
   </link>
@@ -92,10 +92,10 @@
     <visual>
       <origin xyz="0 0 0"/>
-      <geometry><mesh filename="package://mobile_robot/meshes/left_wheel_link.STL"/></geometry>
+      <geometry><mesh filename="package://mobile_robot_description/meshes/left_wheel_link.STL"/></geometry>
       <material name=""><color rgba="0 0 0 1"/></material>
     </visual>
     <collision>
       <origin xyz="0 0 0"/>
-      <geometry><mesh filename="package://mobile_robot/meshes/left_wheel_link.STL"/></geometry>
+      <geometry><mesh filename="package://mobile_robot_description/meshes/left_wheel_link.STL"/></geometry>
     </collision>
   </link>
@@ -119,10 +119,10 @@
     <visual>
       <origin xyz="0 0 0"/>
-      <geometry><mesh filename="package://mobile_robot/meshes/right_wheel_link.STL"/></geometry>
+      <geometry><mesh filename="package://mobile_robot_description/meshes/right_wheel_link.STL"/></geometry>
       <material name=""><color rgba="0.79 0.82 0.93 1"/></material>
     </visual>
     <collision>
       <origin xyz="0 0 0"/>
-      <geometry><mesh filename="package://mobile_robot/meshes/right_wheel_link.STL"/></geometry>
+      <geometry><mesh filename="package://mobile_robot_description/meshes/right_wheel_link.STL"/></geometry>
     </collision>
   </link>
@@ -147,10 +147,10 @@
     <visual>
       <origin xyz="0 0 0"/>
-      <geometry><mesh filename="package://mobile_robot/meshes/lidar.STL"/></geometry>
+      <geometry><mesh filename="package://mobile_robot_description/meshes/lidar.STL"/></geometry>
       <material name=""><color rgba="1 1 1 1"/></material>
     </visual>
     <collision>
       <origin xyz="0 0 0"/>
-      <geometry><mesh filename="package://mobile_robot/meshes/lidar.STL"/></geometry>
+      <geometry><mesh filename="package://mobile_robot_description/meshes/lidar.STL"/></geometry>
     </collision>
   </link>

Commit message: Fix mesh path resolution in Gazebo by switching to $(find ...) URIs

File: mobile_robot_description/urdf/mobile_robot.urdf.xacro (robot description, xacro)
@@ -26,5 +26,5 @@
     <visual>
       <origin xyz="0 0 0" rpy="0 0 0"/>
-      <geometry><mesh filename="package://mobile_robot_description/meshes/chassis.STL"/></geometry>
+      <geometry><mesh filename="$(find mobile_robot_description)/meshes/chassis.STL"/></geometry>
       <material name=""><color rgba="0.647 0.620 0.588 1"/></material>
     </visual>
@@ -32,5 +32,5 @@
     <collision>
       <origin xyz="0 0 0" rpy="0 0 0"/>
-      <geometry><mesh filename="package://mobile_robot_description/meshes/chassis.STL"/></geometry>
+      <geometry><mesh filename="$(find mobile_robot_description)/meshes/chassis.STL"/></geometry>
     </collision>
   </link>
@@ -92,10 +92,10 @@
     <visual>
       <origin xyz="0 0 0"/>
-      <geometry><mesh filename="package://mobile_robot_description/meshes/left_wheel_link.STL"/></geometry>
+      <geometry><mesh filename="$(find mobile_robot_description)/meshes/left_wheel_link.STL"/></geometry>
       <material name=""><color rgba="0 0 0 1"/></material>
     </visual>
     <collision>
       <origin xyz="0 0 0"/>
-      <geometry><mesh filename="package://mobile_robot_description/meshes/left_wheel_link.STL"/></geometry>
+      <geometry><mesh filename="$(find mobile_robot_description)/meshes/left_wheel_link.STL"/></geometry>
     </collision>
   </link>
@@ -119,10 +119,10 @@
     <visual>
       <origin xyz="0 0 0"/>
-      <geometry><mesh filename="package://mobile_robot_description/meshes/right_wheel_link.STL"/></geometry>
+      <geometry><mesh filename="$(find mobile_robot_description)/meshes/right_wheel_link.STL"/></geometry>
       <material name=""><color rgba="0.79 0.82 0.93 1"/></material>
     </visual>
     <collision>
       <origin xyz="0 0 0"/>
-      <geometry><mesh filename="package://mobile_robot_description/meshes/right_wheel_link.STL"/></geometry>
+      <geometry><mesh filename="$(find mobile_robot_description)/meshes/right_wheel_link.STL"/></geometry>
     </collision>
   </link>
@@ -156,10 +156,10 @@
     <visual>
       <origin xyz="0 0 0"/>
-      <geometry><mesh filename="package://mobile_robot_description/meshes/lidar.STL"/></geometry>
+      <geometry><mesh filename="$(find mobile_robot_description)/meshes/lidar.STL"/></geometry>
       <material name=""><color rgba="1 1 1 1"/></material>
     </visual>
     <collision>
       <origin xyz="0 0 0"/>
-      <geometry><mesh filename="package://mobile_robot_description/meshes/lidar.STL"/></geometry>
+      <geometry><mesh filename="$(find mobile_robot_description)/meshes/lidar.STL"/></geometry>
     </collision>
   </link>

Commit message: Fix URDF mesh paths for Gazebo and RViz2
Changed mesh references to use file:// prefix
so that both Gazebo and RViz2 can correctly load STL files.

File: mobile_robot_description/urdf/mobile_robot.urdf.xacro (robot description, xacro)
@@ -26,5 +26,5 @@
     <visual>
       <origin xyz="0 0 0" rpy="0 0 0"/>
-      <geometry><mesh filename="$(find mobile_robot_description)/meshes/chassis.STL"/></geometry>
+      <geometry><mesh filename="file://$(find mobile_robot_description)/meshes/chassis.STL"/></geometry>
       <material name=""><color rgba="0.647 0.620 0.588 1"/></material>
     </visual>
@@ -32,5 +32,5 @@
     <collision>
       <origin xyz="0 0 0" rpy="0 0 0"/>
-      <geometry><mesh filename="$(find mobile_robot_description)/meshes/chassis.STL"/></geometry>
+      <geometry><mesh filename="file://$(find mobile_robot_description)/meshes/chassis.STL"/></geometry>
     </collision>
   </link>
@@ -92,10 +92,10 @@
     <visual>
       <origin xyz="0 0 0"/>
-      <geometry><mesh filename="$(find mobile_robot_description)/meshes/left_wheel_link.STL"/></geometry>
+      <geometry><mesh filename="file://$(find mobile_robot_description)/meshes/left_wheel_link.STL"/></geometry>
       <material name=""><color rgba="0 0 0 1"/></material>
     </visual>
     <collision>
       <origin xyz="0 0 0"/>
-      <geometry><mesh filename="$(find mobile_robot_description)/meshes/left_wheel_link.STL"/></geometry>
+      <geometry><mesh filename="file://$(find mobile_robot_description)/meshes/left_wheel_link.STL"/></geometry>
     </collision>
   </link>
@@ -119,10 +119,10 @@
     <visual>
       <origin xyz="0 0 0"/>
-      <geometry><mesh filename="$(find mobile_robot_description)/meshes/right_wheel_link.STL"/></geometry>
+      <geometry><mesh filename="file://$(find mobile_robot_description)/meshes/right_wheel_link.STL"/></geometry>
       <material name=""><color rgba="0.79 0.82 0.93 1"/></material>
     </visual>
     <collision>
       <origin xyz="0 0 0"/>
-      <geometry><mesh filename="$(find mobile_robot_description)/meshes/right_wheel_link.STL"/></geometry>
+      <geometry><mesh filename="file://$(find mobile_robot_description)/meshes/right_wheel_link.STL"/></geometry>
     </collision>
   </link>
@@ -156,10 +156,10 @@
     <visual>
       <origin xyz="0 0 0"/>
-      <geometry><mesh filename="$(find mobile_robot_description)/meshes/lidar.STL"/></geometry>
+      <geometry><mesh filename="file://$(find mobile_robot_description)/meshes/lidar.STL"/></geometry>
       <material name=""><color rgba="1 1 1 1"/></material>
     </visual>
     <collision>
       <origin xyz="0 0 0"/>
-      <geometry><mesh filename="$(find mobile_robot_description)/meshes/lidar.STL"/></geometry>
+      <geometry><mesh filename="file://$(find mobile_robot_description)/meshes/lidar.STL"/></geometry>
     </collision>
   </link>

Commit message: mobile_robot_web: resolve named material refs in URDF parser
The URDF allows <material name=X/> to reference a top-level
<material name=X><color/></material> definition. The 3D view's
parser was only reading inline <color> tags, so wheels using the
new named black reference fell back to default gray. Build a
registry of top-level material defs first, then look up the name
when a visual's material has no inline color.

File: mobile_robot_description/urdf/mobile_robot.urdf.xacro (robot description, xacro)
@@ -93,5 +93,5 @@
       <origin xyz="0 0 0"/>
       <geometry><mesh filename="file://$(find mobile_robot_description)/meshes/left_wheel_link.STL"/></geometry>
-      <material name=""><color rgba="0 0 0 1"/></material>
+      <material name="black"></material>
     </visual>
     <collision>
@@ -120,5 +120,5 @@
       <origin xyz="0 0 0"/>
       <geometry><mesh filename="file://$(find mobile_robot_description)/meshes/right_wheel_link.STL"/></geometry>
-      <material name=""><color rgba="0.79 0.82 0.93 1"/></material>
+      <material name="black"></material>
     </visual>
     <collision>

Commit message: mobile_robot_web: render URDF sphere/box/cylinder primitives in 3D view
Casters and any other links using URDF primitive geometries
(<sphere>, <box>, <cylinder>) were invisible because the parser only
handled <mesh>. Extract geometry parsing into parseGeometry() and
dispatch to the matching THREE.*Geometry in buildLinkObject. Cylinder
gets a 90° X rotation to convert from URDF's +Z axis to three.js's +Y.
Also honors <mesh scale=...> which was previously ignored.

File: mobile_robot_description/urdf/mobile_robot.urdf.xacro (robot description, xacro)
@@ -51,4 +51,5 @@
         <origin xyz="0 0 0" rpy="0 0 0"/>
         <geometry><sphere radius="0.03"/></geometry>
+        <material name="black"></material>
       </visual>
       <collision>
