Commit message: mobile_robot_description: extract the color into named material
Define the color "grayish-brown" once in materials.xacro and
reference it from the chassis link instead of inlining the RGBA value.
Refer to the white color instead of hardcoding it.

File: mobile_robot_description/urdf/materials.xacro (robot description, xacro)
@@ -13,4 +13,7 @@
     <color rgba="0.2 0.2 0.2 1.0"/>
   </material>
+  <material name="grayish-brown">
+    <color rgba="0.647 0.620 0.588 1"/>
+  </material>
   <material name="orange">
     <color rgba="${255/255} ${108/255} ${10/255} 1.0"/>

File: mobile_robot_description/urdf/mobile_robot.urdf.xacro (robot description, xacro)
@@ -27,5 +27,5 @@
       <origin xyz="0 0 0" rpy="0 0 0"/>
       <geometry><mesh filename="file://$(find mobile_robot_description)/meshes/chassis.STL"/></geometry>
-      <material name=""><color rgba="0.647 0.620 0.588 1"/></material>
+      <material name="grayish-brown"></material>
     </visual>
     <!-- Chassis Collision -->
@@ -158,5 +158,5 @@
       <origin xyz="0 0 0"/>
       <geometry><mesh filename="file://$(find mobile_robot_description)/meshes/lidar.STL"/></geometry>
-      <material name=""><color rgba="1 1 1 1"/></material>
+      <material name="white"></material>
     </visual>
     <collision>
